File: PCB/CosmicGirl.kicad_pcb (KiCad board)
At the start: 2 copper layers, 98 x 98 mm, 35 parts, among them J1 OLED_DISPLAY, M3-1 MountingHole, M3-2 MountingHole, M3-3 MountingHole, M3-4 MountingHole, SW1 SW_Push, SW10 RotaryEncoder_Switch, SW2 SW_Push, SW3 SW_Push, SW4 SW_Push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

Commit message: Update
Connections:
- SW10 pad S2: COL2 -> ROW0
Routing:
- net ROW0: track 129.9 -> 169.0 mm
- net COL2: track 155.6 -> 158.1 mm, vias 2 -> 4
