File: PCB/CosmicGirl.kicad_sch (KiCad schematic)
At the start: 35 parts, among them J1 OLED_DISPLAY, M3-1 MountingHole, M3-2 MountingHole, M3-3 MountingHole, M3-4 MountingHole, SW1 SW_Push, SW10 RotaryEncoder_Switch, SW2 SW_Push, SW3 SW_Push, SW4 SW_Push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

Commit message: Update
Connections:
- net COL2: no longer SW10.S2
- net ROW0: now also SW10.S2
Changed lines of the file:
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@@
 		)
 	)
-	(global_label "COL2"
+	(global_label "ROW0"
 		(shape input)
 		(at 58.42 36.83 180)
@@
 		)
 		(instances
-			(project "3x3 macropad"
+			(project "CosmicGirl"
 				(path "/b549fe80-d2b1-4469-a6fa-02c0072a15ad"
 					(reference "SW1")
@@
 		)
 		(instances
-			(project "3x3 macropad"
+			(project "CosmicGirl"
 				(path "/b549fe80-d2b1-4469-a6fa-02c0072a15ad"
 					(reference "M3-4")
@@
 		)
 		(instances
-			(project "3x3 macropad"
+			(project "CosmicGirl"
 				(path "/b549fe80-d2b1-4469-a6fa-02c0072a15ad"
 					(reference "M3-3")
@@
 		)
 		(instances
-			(project "3x3 macropad"
+			(project "CosmicGirl"
 				(path "/b549fe80-d2b1-4469-a6fa-02c0072a15ad"
 					(reference "D16")
@@
 		)
 		(instances
-			(project "3x3 macropad"
+			(project "CosmicGirl"
 				(path "/b549fe80-d2b1-4469-a6fa-02c0072a15ad"
 					(reference "D17")
@@
 		)
 		(instances
-			(project "3x3 macropad"
+			(project "CosmicGirl"
 				(path "/b549fe80-d2b1-4469-a6fa-02c0072a15ad"
 					(reference "#PWR08")
@@
 		)
 		(instances
-			(project "3x3 macropad"
+			(project "CosmicGirl"
 				(path "/b549fe80-d2b1-4469-a6fa-02c0072a15ad"
 					(reference "D4")
@@
 		)
 		(instances
-			(project "3x3 macropad"
+			(project "CosmicGirl"
 				(path "/b549fe80-d2b1-4469-a6fa-02c0072a15ad"
 					(reference "M3-2")
@@
 		)
 		(instances
-			(project "3x3 macropad"
+			(project "CosmicGirl"
 				(path "/b549fe80-d2b1-4469-a6fa-02c0072a15ad"
 					(reference "D1")
@@
 		)
 		(instances
-			(project "3x3 macropad"
+			(project "CosmicGirl"
 				(path "/b549fe80-d2b1-4469-a6fa-02c0072a15ad"
 					(reference "#PWR06")
@@
 		)
 		(instances
-			(project "3x3 macropad"
+			(project "CosmicGirl"
 				(path "/b549fe80-d2b1-4469-a6fa-02c0072a15ad"
 					(reference "#PWR011")
@@
 		)
 		(instances
-			(project "3x3 macropad"
+			(project "CosmicGirl"
 				(path "/b549fe80-d2b1-4469-a6fa-02c0072a15ad"
 					(reference "SW8")
@@
 		)
 		(instances
-			(project "3x3 macropad"
+			(project "CosmicGirl"
 				(path "/b549fe80-d2b1-4469-a6fa-02c0072a15ad"
 					(reference "#PWR013")
@@
 		)
 		(instances
-			(project "3x3 macropad"
+			(project "CosmicGirl"
 				(path "/b549fe80-d2b1-4469-a6fa-02c0072a15ad"
 					(reference "#PWR01")
@@
 		)
 		(instances
-			(project "3x3 macropad"
+			(project "CosmicGirl"
 				(path "/b549fe80-d2b1-4469-a6fa-02c0072a15ad"
 					(reference "D15")
@@
 		)
 		(instances
-			(project "3x3 macropad"
+			(project "CosmicGirl"
 				(path "/b549fe80-d2b1-4469-a6fa-02c0072a15ad"
 					(reference "D12")
@@
 		)
 		(instances
-			(project "3x3 macropad"
+			(project "CosmicGirl"
 				(path "/b549fe80-d2b1-4469-a6fa-02c0072a15ad"
 					(reference "#PWR03")
@@
 		)
 		(instances
-			(project "3x3 macropad"
+			(project "CosmicGirl"
 				(path "/b549fe80-d2b1-4469-a6fa-02c0072a15ad"
 					(reference "D7")
@@
 		)
 		(instances
-			(project "3x3 macropad"
+			(project "CosmicGirl"
 				(path "/b549fe80-d2b1-4469-a6fa-02c0072a15ad"
 					(reference "SW10")
@@
 		)
 		(instances
-			(project "3x3 macropad"
+			(project "CosmicGirl"
 				(path "/b549fe80-d2b1-4469-a6fa-02c0072a15ad"
 					(reference "D9")
@@
 		)
 		(instances
-			(project "3x3 macropad"
+			(project "CosmicGirl"
 				(path "/b549fe80-d2b1-4469-a6fa-02c0072a15ad"
 					(reference "J1")
@@
 		)
 		(instances
-			(project "3x3 macropad"
+			(project "CosmicGirl"
 				(path "/b549fe80-d2b1-4469-a6fa-02c0072a15ad"
 					(reference "D13")
@@
 		)
 		(instances
-			(project "3x3 macropad"
+			(project "CosmicGirl"
 				(path "/b549fe80-d2b1-4469-a6fa-02c0072a15ad"
 					(reference "SW6")
@@
 		)
 		(instances
-			(project "3x3 macropad"
+			(project "CosmicGirl"
 				(path "/b549fe80-d2b1-4469-a6fa-02c0072a15ad"
 					(reference "M3-1")
@@
 		)
 		(instances
-			(project "3x3 macropad"
+			(project "CosmicGirl"
 				(path "/b549fe80-d2b1-4469-a6fa-02c0072a15ad"
 					(reference "#PWR09")
@@
 		)
 		(instances
-			(project "3x3 macropad"
+			(project "CosmicGirl"
 				(path "/b549fe80-d2b1-4469-a6fa-02c0072a15ad"
 					(reference "D11")
@@
 		)
 		(instances
-			(project "3x3 macropad"
+			(project "CosmicGirl"
 				(path "/b549fe80-d2b1-4469-a6fa-02c0072a15ad"
 					(reference "#PWR05")
@@
 		)
 		(instances
-			(project "3x3 macropad"
+			(project "CosmicGirl"
 				(path "/b549fe80-d2b1-4469-a6fa-02c0072a15ad"
 					(reference "D6")
@@
 		)
 		(instances
-			(project "3x3 macropad"
+			(project "CosmicGirl"
 				(path "/b549fe80-d2b1-4469-a6fa-02c0072a15ad"
 					(reference "SW7")
@@
 		)
 		(instances
-			(project "3x3 macropad"
+			(project "CosmicGirl"
 				(path "/b549fe80-d2b1-4469-a6fa-02c0072a15ad"
 					(reference "D14")
@@
 		)
 		(instances
-			(project "3x3 macropad"
+			(project "CosmicGirl"
 				(path "/b549fe80-d2b1-4469-a6fa-02c0072a15ad"
 					(reference "#PWR019")
@@
 		)
 		(instances
-			(project "3x3 macropad"
+			(project "CosmicGirl"
 				(path "/b549fe80-d2b1-4469-a6fa-02c0072a15ad"
 					(reference "U1")
@@
 		)
 		(instances
-			(project "3x3 macropad"
+			(project "CosmicGirl"
 				(path "/b549fe80-d2b1-4469-a6fa-02c0072a15ad"
 					(reference "D5")
@@
 		)
 		(instances
-			(project "3x3 macropad"
+			(project "CosmicGirl"
 				(path "/b549fe80-d2b1-4469-a6fa-02c0072a15ad"
 					(reference "SW4")
@@
 		)
 		(instances
-			(project "3x3 macropad"
+			(project "CosmicGirl"
 				(path "/b549fe80-d2b1-4469-a6fa-02c0072a15ad"
 					(reference "SW5")
@@
 		)
 		(instances
-			(project "3x3 macropad"
+			(project "CosmicGirl"
 				(path "/b549fe80-d2b1-4469-a6fa-02c0072a15ad"
 					(reference "#PWR012")
@@
 		)
 		(instances
-			(project "3x3 macropad"
+			(project "CosmicGirl"
 				(path "/b549fe80-d2b1-4469-a6fa-02c0072a15ad"
 					(reference "D2")
@@
 		)
 		(instances
-			(project "3x3 macropad"
+			(project "CosmicGirl"
 				(path "/b549fe80-d2b1-4469-a6fa-02c0072a15ad"
 					(reference "#PWR016")
@@
 		)
 		(instances
-			(project "3x3 macropad"
+			(project "CosmicGirl"
 				(path "/b549fe80-d2b1-4469-a6fa-02c0072a15ad"
 					(reference "#PWR021")
@@
 		)
 		(instances
-			(project "3x3 macropad"
+			(project "CosmicGirl"
 				(path "/b549fe80-d2b1-4469-a6fa-02c0072a15ad"
 					(reference "D18")
@@
 		)
 		(instances
-			(project "3x3 macropad"
+			(project "CosmicGirl"
 				(path "/b549fe80-d2b1-4469-a6fa-02c0072a15ad"
 					(reference "#PWR02")
@@
 		)
 		(instances
-			(project "3x3 macropad"
+			(project "CosmicGirl"
 				(path "/b549fe80-d2b1-4469-a6fa-02c0072a15ad"
 					(reference "D10")
@@
 		)
 		(instances
-			(project "3x3 macropad"
+			(project "CosmicGirl"
 				(path "/b549fe80-d2b1-4469-a6fa-02c0072a15ad"
 					(reference "D19")
@@
 		)
 		(instances
-			(project "3x3 macropad"
+			(project "CosmicGirl"
 				(path "/b549fe80-d2b1-4469-a6fa-02c0072a15ad"
 					(reference "#PWR04")
@@
 		)
 		(instances
-			(project "3x3 macropad"
+			(project "CosmicGirl"
 				(path "/b549fe80-d2b1-4469-a6fa-02c0072a15ad"
 					(reference "SW9")
@@
 		)
 		(instances
-			(project "3x3 macropad"
+			(project "CosmicGirl"
 				(path "/b549fe80-d2b1-4469-a6fa-02c0072a15ad"
 					(reference "#PWR07")
@@
 		)
 		(instances
-			(project "3x3 macropad"
+			(project "CosmicGirl"
 				(path "/b549fe80-d2b1-4469-a6fa-02c0072a15ad"
 					(reference "SW3")
@@
 		)
 		(instances
-			(project "3x3 macropad"
+			(project "CosmicGirl"
 				(path "/b549fe80-d2b1-4469-a6fa-02c0072a15ad"
 					(reference "#PWR014")
@@
 		)
 		(instances
-			(project "3x3 macropad"
+			(project "CosmicGirl"
 				(path "/b549fe80-d2b1-4469-a6fa-02c0072a15ad"
 					(reference "D3")
@@
 		)
 		(instances
-			(project "3x3 macropad"
+			(project "CosmicGirl"
 				(path "/b549fe80-d2b1-4469-a6fa-02c0072a15ad"
 					(reference "SW2")
@@
 		)
 		(instances
-			(project "3x3 macropad"
+			(project "CosmicGirl"
 				(path "/b549fe80-d2b1-4469-a6fa-02c0072a15ad"
 					(reference "#PWR010")
@@
 		)
 		(instances
-			(project "3x3 macropad"
+			(project "CosmicGirl"
 				(path "/b549fe80-d2b1-4469-a6fa-02c0072a15ad"
 					(reference "#PWR018")
@@
 		)
 		(instances
-			(project "3x3 macropad"
+			(project "CosmicGirl"
 				(path "/b549fe80-d2b1-4469-a6fa-02c0072a15ad"
 					(reference "D8")
@@
 		)
 		(instances
-			(project "3x3 macropad"
+			(project "CosmicGirl"
 				(path "/b549fe80-d2b1-4469-a6fa-02c0072a15ad"
 					(reference "#PWR015")
@@
 		)
 		(instances
-			(project "3x3 macropad"
+			(project "CosmicGirl"
 				(path "/b549fe80-d2b1-4469-a6fa-02c0072a15ad"
 					(reference "#PWR017")
@@
 		)
 		(instances
-			(project "3x3 macropad"
+			(project "CosmicGirl"
 				(path "/b549fe80-d2b1-4469-a6fa-02c0072a15ad"
 					(reference "#PWR020")
